File: irisc.sch (EAGLE design)
At the start: 0 parts

Commit message: RPI
Parts:
- added X1: RASPI_BOARD_B+_E4, raspberrypi_bastelstube_v13:RASPI_BOARD_B+_E4
Changed lines of the file:
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@@
 <layers>
 <layer number="1" name="Top" color="4" fill="1" visible="no" active="no"/>
+<layer number="2" name="Route2" color="1" fill="3" visible="no" active="no"/>
+<layer number="3" name="Route3" color="4" fill="3" visible="no" active="no"/>
+<layer number="4" name="Route4" color="1" fill="4" visible="no" active="no"/>
+<layer number="5" name="Route5" color="4" fill="4" visible="no" active="no"/>
+<layer number="6" name="Route6" color="1" fill="8" visible="no" active="no"/>
+<layer number="7" name="Route7" color="4" fill="8" visible="no" active="no"/>
+<layer number="8" name="Route8" color="1" fill="2" visible="no" active="no"/>
+<layer number="9" name="Route9" color="4" fill="2" visible="no" active="no"/>
+<layer number="10" name="Route10" color="1" fill="7" visible="no" active="no"/>
+<layer number="11" name="Route11" color="4" fill="7" visible="no" active="no"/>
+<layer number="12" name="Route12" color="1" fill="5" visible="no" active="no"/>
+<layer number="13" name="Route13" color="4" fill="5" visible="no" active="no"/>
+<layer number="14" name="Route14" color="1" fill="6" visible="no" active="no"/>
+<layer number="15" name="Route15" color="4" fill="6" visible="no" active="no"/>
 <layer number="16" name="Bottom" color="1" fill="1" visible="no" active="no"/>
 <layer number="17" name="Pads" color="2" fill="1" visible="no" active="no"/>
@@
 <parts>
 <part name="FRAME1" library="frames" library_urn="urn:adsk.eagle:library:229" deviceset="A4L-LOC" device=""/>
+<part name="X1" library="raspberrypi_bastelstube_v13" deviceset="RASPI_BOARD_B+" device="_E4"/>
 </parts>
 <sheets>
@@
 <attribute name="SHEET" x="555.625" y="-220.98" size="2.54" layer="94"/>
 </instance>
+<instance part="X1" gate="G$1" x="414.02" y="-111.76" smashed="yes"/>
 </instances>
 <busses>

Commit message: Update irisc.sch
Parts:
- added BUCK_CONVERTER1, U1: LM2695MH, LM2695MH:LM2695MH
- added C1, C2: (no value), Wurth_Elektronik_Passive_Capacitors_rev18b:WCAP-CSGP_0805_885012006082_REFLOW
- added C10, C11, C12, C13, C14, C15, C16, C17, C18, C19, C3, C4, C5, C6, C7, C8, C9: (no value), Wurth_Elektronik_Passive_Capacitors_rev18b:WCAP-CSGP_0805_885012006018_WAVE
- added D1: (no value), BeagleBone_Blue_R3:DIODE
- added L1, L2, L3: (no value), BeagleBone_Blue_R3:INDUCTOR
- added R1, R10, R11, R12, R13, R2, R3, R4, R5, R6, R7, R8, R9: (no value), adafruit:FLIPFLOP-RES
- added U2: (no value), SOP65P640X120-17N:BUCK_CONVERTER1
- added U3: BUCK_CONVERTER2, SOIC127P600X170-8N:BUCK_CONVERTER2
Connections:
- new net 0: BUCK_CONVERTER1.FB, BUCK_CONVERTER1.SGND, C1.1, C10.1, C14.1, C15.1, C18.1, C19.1, C2.1, C3.1, C4.1, C6.1, C8.1, R13.2, R4.1, R6.1, R7.1, U2.AGND, U2.SYNC, U3.AGND, U3.PGND1
- new net 12V: L1.2, R2.2, R3.2
- new net 3.3V: C10.2, C11.2, C12.1, C13.1, C13.2, L2.2, R10.1, R8.2, U2.BIAS, U2.PGND1, U2.PGND2
- new net 5V: C17.2, C18.2, L3.2, R12.1
- new net N$11: C6.2, R3.1
- new net N$12: C7.1, U2.EN
- new net N$13: R5.1, R6.2
- new net N$14: C8.2, U2.SS/TRK
- new net N$15: R7.2, U2.RT
- new net N$16: C12.2, U2.VCC
- new net N$17: C9.2, L2.1, U2.SW1, U2.SW2
- new net N$18: C9.1, U2.CBOOT
- new net N$2: BUCK_CONVERTER1.RON/SD, R1.1
- new net N$20: C11.1, R8.1, R9.2, U2.FB
- new net N$21: R10.2, U2.PGOOD
- new net N$23: C19.2, R11.1, U3.VCC
- new net N$24: R11.2, U3.PG
- new net N$25: C16.2, U3.BOOT
- new net N$26: C16.1, L3.1, U3.SW
- new net N$29: C17.1, R12.2, R13.1, U3.FB
- new net N$3: BUCK_CONVERTER1.SS, C3.2
- new net N$4: BUCK_CONVERTER1.RTN, R2.1, R4.2
- new net N$6: BUCK_CONVERTER1.VCC, C4.2
- new net N$7: BUCK_CONVERTER1.BST, C5.2
- new net N$8: BUCK_CONVERTER1.SW, C5.1, D1.C, L1.1
- new net N$9: BUCK_CONVERTER1.ISEN, D1.A
- new net VCC: BUCK_CONVERTER1.VIN, C1.2, C14.2, C15.2, C2.2, C7.2, R1.2, R5.2, U2.VIN1, U2.VIN2, U3.EN, U3.VIN1
Other:
- note added: "Buck converter: LM2695MH"
- note added: "Buck converter: LM43600PWPR"
- note added: "Buck conveter: LMR33630ADDA"

Commit message: Update irisc.sch
Parts:
- added IC1: L298, st-microelectronics:L298
- added U4: PCA9685, SparkFun-IC-Special-Function:PCA9685
- added X2: RASPI_BOARD_B+_E4, raspberrypi_bastelstube_v13:RASPI_BOARD_B+_E4
Connections:
- new net N$1: U4.SDA, X2.SDA
- new net N$10: IC1.INPUT4, X2.SPI_CE1
- new net N$19: IC1.INPUT3, X2.SPI_CE0
- new net N$22: IC1.INPUT2, X2.SPI_MISO
- new net N$27: IC1.INPUT1, X2.SPI_MOSI
- new net N$5: U4.SCL, X2.SCL
- net 0: now also IC1.GND, X2.GND
- net VCC: now also X2.5V0
Changed lines of the file:
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@@
 <part name="SUPPLY3" library="SparkFun-PowerSymbols" library_urn="urn:adsk.eagle:library:530" deviceset="5V" device=""/>
 <part name="SUPPLY4" library="SparkFun-PowerSymbols" library_urn="urn:adsk.eagle:library:530" deviceset="3.3V" device=""/>
+<part name="FRAME3" library="frames" library_urn="urn:adsk.eagle:library:229" deviceset="A4L-LOC" device=""/>
+<part name="X2" library="raspberrypi_bastelstube_v13" deviceset="RASPI_BOARD_B+" device="_E4"/>
+<part name="U4" library="SparkFun-IC-Special-Function" library_urn="urn:adsk.eagle:library:527" deviceset="PCA9685" device="" package3d_urn="urn:adsk.eagle:package:39196/1" value="PCA9685"/>
+<part name="IC1" library="st-microelectronics" library_urn="urn:adsk.eagle:library:368" deviceset="L298" device="" package3d_urn="urn:adsk.eagle:package:26823/1"/>
+<part name="X_10" library="ngspice-simulation" library_urn="urn:adsk.eagle:library:527439" deviceset="GND" device=""/>
+<part name="X_11" library="ngspice-simulation" library_urn="urn:adsk.eagle:library:527439" deviceset="GND" device=""/>
+<part name="P+1" library="audio amplifier example" library_urn="urn:adsk.eagle:library:970892" deviceset="VCC" device=""/>
 </parts>
 <sheets>
@@
 </segment>
 </net>
+</nets>
+</sheet>
+<sheet>
+<plain>
+</plain>
+<instances>
+<instance part="FRAME3" gate="G$1" x="0" y="0" smashed="yes">
+<attribute name="DRAWING_NAME" x="217.17" y="15.24" size="2.54" layer="94"/>
+<attribute name="LAST_DATE_TIME" x="217.17" y="10.16" size="2.286" layer="94"/>
+<attribute name="SHEET" x="230.505" y="5.08" size="2.54" layer="94"/>
+</instance>
+<instance part="X2" gate="G$1" x="35.56" y="139.7" smashed="yes"/>
+<instance part="U4" gate="G$1" x="83.82" y="124.46" smashed="yes">
+<attribute name="NAME" x="83.82" y="165.1" size="1.778" layer="95"/>
+<attribute name="VALUE" x="83.82" y="163.068" size="1.778" layer="96"/>
+</instance>
+<instance part="IC1" gate="L298" x="149.86" y="142.24" smashed="yes">
+<attribute name="NAME" x="137.16" y="161.29" size="1.778" layer="95"/>
+<attribute name="VALUE" x="137.16" y="127" size="1.778" layer="96"/>
+</instance>
+<instance part="X_10" gate="G$1" x="35.56" y="99.06" smashed="yes"/>
+<instance part="X_11" gate="G$1" x="132.08" y="127" smashed="yes"/>
+<instance part="P+1" gate="VCC" x="30.48" y="172.72" smashed="yes">
+<attribute name="VALUE" x="28.956" y="173.736" size="1.27" layer="96"/>
+</instance>
+</instances>
+<busses>
+</busses>
+<nets>
+<net name="N$1" class="0">
+<segment>
+<pinref part="X2" gate="G$1" pin="SDA"/>
+<wire x1="20.32" y1="104.14" x2="15.24" y2="104.14" width="0.1524" layer="91"/>
+<wire x1="15.24" y1="104.14" x2="15.24" y2="96.52" width="0.1524" layer="91"/>
+<wire x1="15.24" y1="96.52" x2="71.12" y2="96.52" width="0.1524" layer="91"/>
+<wire x1="71.12" y1="96.52" x2="71.12" y2="167.64" width="0.1524" layer="91"/>
+<wire x1="71.12" y1="167.64" x2="111.76" y2="167.64" width="0.1524" layer="91"/>
+<wire x1="111.76" y1="167.64" x2="111.76" y2="157.48" width="0.1524" layer="91"/>
+<pinref part="U4" gate="G$1" pin="SDA"/>
+<wire x1="111.76" y1="157.48" x2="106.68" y2="157.48" width="0.1524" layer="91"/>
+</segment>
+</net>
+<net name="N$5" class="0">
+<segment>
+<pinref part="X2" gate="G$1" pin="SCL"/>
+<wire x1="20.32" y1="106.68" x2="12.7" y2="106.68" width="0.1524" layer="91"/>
+<wire x1="12.7" y1="106.68" x2="12.7" y2="93.98" width="0.1524" layer="91"/>
+<wire x1="12.7" y1="93.98" x2="73.66" y2="93.98" width="0.1524" layer="91"/>
+<wire x1="73.66" y1="93.98" x2="73.66" y2="165.1" width="0.1524" layer="91"/>
+<wire x1="73.66" y1="165.1" x2="109.22" y2="165.1" width="0.1524" layer="91"/>
+<wire x1="109.22" y1="165.1" x2="109.22" y2="154.94" width="0.1524" layer="91"/>
+<pinref part="U4" gate="G$1" pin="SCL"/>
+<wire x1="109.22" y1="154.94" x2="106.68" y2="154.94" width="0.1524" layer="91"/>
+</segment>
+</net>
+<net name="0" class="0">
+<segment>
+<pinref part="X2" gate="G$1" pin="GND"/>
+<pinref part="X_10" gate="G$1" pin="0"/>
+</segment>
+<segment>
+<pinref part="IC1" gate="L298" pin="GND"/>
+<wire x1="134.62" y1="132.08" x2="132.08" y2="132.08" width="0.1524" layer="91"/>
+<pinref part="X_11" gate="G$1" pin="0"/>
+<wire x1="132.08" y1="132.08" x2="132.08" y2="127" width="0.1524" layer="91"/>
+</segment>
+</net>
+<net name="VCC" class="0">
+<segment>
+<pinref part="X2" gate="G$1" pin="5V0"/>
+<wire x1="30.48" y1="167.64" x2="30.48" y2="170.18" width="0.1524" layer="91"/>
+<pinref part="P+1" gate="VCC" pin="VCC"/>
+</segment>
+</net>
+<net name="N$10" class="0">
+<segment>
+<pinref part="X2" gate="G$1" pin="SPI_CE1"/>
+<wire x1="50.8" y1="144.78" x2="60.96" y2="144.78" width="0.1524" layer="91"/>
+<wire x1="60.96" y1="144.78" x2="60.96" y2="106.68" width="0.1524" layer="91"/>
+<wire x1="60.96" y1="106.68" x2="127" y2="106.68" width="0.1524" layer="91"/>
+<wire x1="127" y1="106.68" x2="127" y2="137.16" width="0.1524" layer="91"/>
+<pinref part="IC1" gate="L298" pin="INPUT4"/>
+<wire x1="127" y1="137.16" x2="134.62" y2="137.16" width="0.1524" layer="91"/>
+</segment>
+</net>
+<net name="N$19" class="0">
+<segment>
+<pinref part="X2" gate="G$1" pin="SPI_CE0"/>
+<wire x1="50.8" y1="147.32" x2="63.5" y2="147.32" width="0.1524" layer="91"/>
+<wire x1="63.5" y1="147.32" x2="63.5" y2="109.22" width="0.1524" layer="91"/>
+<wire x1="63.5" y1="109.22" x2="124.46" y2="109.22" width="0.1524" layer="91"/>
+<pinref part="IC1" gate="L298" pin="INPUT3"/>
+<wire x1="124.46" y1="109.22" x2="124.46" y2="139.7" width="0.1524" layer="91"/>
+<wire x1="124.46" y1="139.7" x2="134.62" y2="139.7" width="0.1524" layer="91"/>
+</segment>
+</net>
+<net name="N$22" class="0">
+<segment>
+<pinref part="X2" gate="G$1" pin="SPI_MISO"/>
+<wire x1="50.8" y1="152.4" x2="66.04" y2="152.4" width="0.1524" layer="91"/>
+<wire x1="66.04" y1="152.4" x2="66.04" y2="111.76" width="0.1524" layer="91"/>
+<wire x1="66.04" y1="111.76" x2="119.38" y2="111.76" width="0.1524" layer="91"/>
+<wire x1="119.38" y1="111.76" x2="119.38" y2="142.24" width="0.1524" layer="91"/>
+<pinref part="IC1" gate="L298" pin="INPUT2"/>
+<wire x1="119.38" y1="142.24" x2="134.62" y2="142.24" width="0.1524" layer="91"/>
+</segment>
+</net>
+<net name="N$27" class="0">
+<segment>
+<pinref part="X2" gate="G$1" pin="SPI_MOSI"/>
+<wire x1="50.8" y1="154.94" x2="68.58" y2="154.94" width="0.1524" layer="91"/>
+<wire x1="68.58" y1="154.94" x2="68.58" y2="114.3" width="0.1524" layer="91"/>
+<wire x1="68.58" y1="114.3" x2="116.84" y2="114.3" width="0.1524" layer="91"/>
+<wire x1="116.84" y1="114.3" x2="116.84" y2="144.78" width="0.1524" layer="91"/>
+<pinref part="IC1" gate="L298" pin="INPUT1"/>
+<wire x1="116.84" y1="144.78" x2="134.62" y2="144.78" width="0.1524" layer="91"/>
+</segment>
+</net>

Commit message: Update motorcontroller, added sensors
Parts:
- removed X2: RASPI_BOARD_B+_E4, raspberrypi_bastelstube_v13:RASPI_BOARD_B+_E4
- added ENCODER@X, ENCODER@Y, ENCODER@Z: (no value), con-amp-mt:L05P
- added IC2: L298, st-microelectronics:L298
- added IC3, IC4, IC5: ADS1271, texas:ADS1271
- added J1: (no value), Wurth_Elektronik_Electromechanic_Coaxial _Connectors_rev18a:60314202124525
- added MOTOR@R, MOTOR@X, MOTOR@Y, MOTOR@Z: (no value), con-amp-mt:L02P
- added SV1: (no value), con-amp-mt:L03P
- added U$1, U$2, U$3, U$4: 100nF, Nordic_nRF:CAPACITOR_0805_L
- added U$5: 1uF, Nordic_nRF:CAPACITOR_0805_L
- added U$6: NEO-M8, ubloxLib:NEO-M8
- added U$7, U$8, U$9: 1uF, Nordic_nRF:CAPACITOR_0603_N
- added U10, U5, U9: ANALOG_DEVICES_ADXRS646BBGZANALOG_DEVICES_ADXRS646BBGZ_0_0, Analog Devices - ADXRS646BBGZ:ANALOG_DEVICES_ADXRS646BBGZANALOG_DEVICES_ADXRS646BBGZ_0_0
- added U6, U8: ANALOG_DEVICES_AD7997BRUZ-1REELANALOG_DEVICES_AD7997BRUZ-1R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, Analog Devices - AD7997BRUZ-1REEL:ANALOG_DEVICES_AD7997BRUZ-1REELANALOG_DEVICES_AD7997BRUZ-1REEL_0_0
- added U7: MELEXIS_TECHNOLOGIES_MLX90393SLW-ABA-011-REMELEXIS_TECHNOLO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, Melexis Technologies - MLX90393SLW-ABA-011-RE:MELEXIS_TECHNOLOGIES_MLX90393SLW-ABA-011-REMELEXIS_TECHNOLOGIES_MLX90393S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
- U1: value LM2695MH -> KXTJ3-1057; device LM2695MH:LM2695MH -> KXTJ3-1057:KXTJ3-1057
Connections:
- new net CE0: X1.SPI_CE0
- new net CE1: X1.SPI_CE1
- new net CLK: ENCODER@X-3.S, ENCODER@Y-3.S, ENCODER@Z-3.S, U$6.19_SCL/SPI_CLK, X1.SPI_SCLK
- new net MISO: ENCODER@X-2.S, ENCODER@Y-2.S, ENCODER@Z-2.S, U$6.20_TXD/SPI_MISO, X1.SPI_MISO
- new net MOSI: U$6.21_RXD/SPI_MOSI, X1.SPI_MOSI
- new net N$28: IC2.INPUT3, U4.CH9
- new net N$30: IC2.INPUT4, U4.CH8
- new net N$31: IC1.OUT1, MOTOR@X-1.S
- new net N$32: IC1.OUT2, MOTOR@X-2.S
- new net N$33: IC1.OUT3, MOTOR@Y-1.S
- new net N$34: IC1.OUT4, MOTOR@Y-2.S
- new net N$35: IC2.OUT1, MOTOR@Z-1.S
- new net N$36: IC2.OUT2, MOTOR@Z-2.S
- new net N$37: IC2.OUT3, MOTOR@R-1.S
- new net N$38: IC2.OUT4, MOTOR@R-2.S
- new net N$39: J1.1, U$6.11_RF_IN
- new net N$41: U$6.18_SDA/SPI_CS_N
- new net N$43: ENCODER@Z-4.S
- new net N$46: ENCODER@X-4.S
- new net N$49: ENCODER@Y-4.S
- new net SCL: U1.SCL, U4.SCL, U7.SCL/SCLK, X1.SCL
- new net SDA: U1.SDA, U4.SDA, U7.SDA/MOSI, X1.SDA
- net 0: now also ENCODER@X-5.S, ENCODER@Y-5.S, ENCODER@Z-5.S, IC1.SEN_A, IC1.SEN_B, IC2.GND, IC2.SEN_A, IC2.SEN_B, J1.2, U$1.2, U$2.1, U$3.2, U$4.1, U$5.2, U$6.10_GND, U$6.12_GND, U$6.13_GND, U$6.24_GND, U$6.2_D_SEL, U$7.1, U$8.2, U$9.2, U1.GND, U1.RES, U4.!OE, U4.A5, U4.EXTCLK, U4.VSS, U7.GND_PAD, U7.VSS, X1.GND; no longer X2.GND
- net 12V: now also IC1.VS, IC2.VS, U$1.1, U$3.1
- net 3.3V: now also U$6.23_VCC, U$7.2, U$8.1, U$9.1, U1.IO_VDD, U1.VDD, U7.VDD, U7.VDD_IO
- net 5V: now also ENCODER@X-1.S, ENCODER@Y-1.S, ENCODER@Z-1.S, IC1.VCC, IC2.VCC, U$2.2, U$4.2, U$5.1, U4.VDD, X1.5V0
- net N$1: now also IC1.INPUT1, U4.CH15; no longer U4.SDA, X2.SDA
- net N$10: now also IC1.INPUT3, U4.CH13; no longer IC1.INPUT4, X2.SPI_CE1
- net N$19: now also IC1.INPUT4, U4.CH12; no longer IC1.INPUT3, X2.SPI_CE0
- net N$22: now also IC2.INPUT1, U4.CH11; no longer IC1.INPUT2, X2.SPI_MISO
- net N$27: now also IC2.INPUT2, U4.CH10; no longer IC1.INPUT1, X2.SPI_MOSI
- net N$5: now also IC1.INPUT2, U4.CH14; no longer U4.SCL, X2.SCL
- net VCC: no longer X2.5V0
Other:
- note added: "Gyroscopes"
- note added: "Motor controller"
- note added: "Power Management"
- note added: "Sensors and onboard computer"
- note added: "Thermal"
