File: irisc.sch (EAGLE design)
At the start: 116 parts, among them IC1 L298, IC2 L298, IC3 ADS1271, IC4 ADS1271, IC5 ADS1271, U1 KXTJ3-1057, U10 ANALOG_DEVICES_ADXRS646BBGZAN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, U3 BUCK_CONVERTER2, U4 PCA9685, U5 ANALOG_DEVICES_ADXRS646BBGZAN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, U6 ANALOG_DEVICES_AD7997BRUZ-1RE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, U7 MELEXIS_TECHNOLOGIES_MLX90393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, U8 ANALOG_DEVICES_AD7997BRUZ-1RE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, U9 ANALOG_DEVICES_ADXRS646BBGZAN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, X1 RASPI_BOARD_B+_E4

Commit message: update embedded
Parts:
- removed BUCKCONVERTER1: (no value), SO-8:BUCK-CONVERTER5V4A
- removed BUCK_CONVERTER2: LM2695MH, LM2695MH:LM2695MH
- removed C20, C21: (no value), Wurth_Elektronik_Passive_Capacitors_rev18b:WCAP-CSGP_0805_885012006082_REFLOW
- removed C22, C23, C24, C25, C26, C27, C28, C29, C30, C31, C32, C33, C34, C35, C36, C37, C38, C39, C40, C41, C42, C43, C44: (no value), Wurth_Elektronik_Passive_Capacitors_rev18b:WCAP-CSGP_0805_885012006018_WAVE
- removed D2: (no value), BeagleBone_Blue_R3:DIODE
- removed IC3, IC4, IC5: ADS1271, texas:ADS1271
- removed L4, L5: (no value), BeagleBone_Blue_R3:INDUCTOR
- removed L6: 22uH, BeagleBone_Blue_R3:INDUCTOR
- removed SV1: (no value), con-amp-mt:L03P
- removed U10, U9: ANALOG_DEVICES_ADXRS646BBGZANALOG_DEVICES_ADXRS646BBGZ_0_0, Analog Devices - ADXRS646BBGZ:ANALOG_DEVICES_ADXRS646BBGZANALOG_DEVICES_ADXRS646BBGZ_0_0
- added FB1, FB2, FB3, FB4: 30Ω/1.8A, SparkFun-Coils:FERRITE_BEAD-0603
- added R16, R30, R32, R34, R38: 100k, SparkFun-Resistors:100KOHM-0603-1/10W-1%
- added R23, R29, R31, R33, R35, R37: 10k, SparkFun-Resistors:100KOHM-0603-1/10W-1%
- added R36: 5.6k, SparkFun-Resistors:5.6KOHM-0603-1/10W-1%
- added SELF-TEST, TEMPA@1, TEMPA@2, TEMPA@3, TEMPA@4, TEMPA@5, TEMPA@6, TEMPA@7, TEMPA@8, TEMPA@9: (no value), con-amp-mt:L02P
- added T1, T2, T3, T4, T5, T6, T7, T8, T9: (no value), DC_LOAD_AU:-PNP-SOT23-BEC
- added T10: (no value), DC_LOAD_AU:-NPN-SOT23-BEC
- added TEMPS@1, TEMPS@10, TEMPS@11, TEMPS@12, TEMPS@13, TEMPS@14, TEMPS@15, TEMPS@16, TEMPS@2, TEMPS@3, TEMPS@4, TEMPS@5, TEMPS@6, TEMPS@7, TEMPS@8, TEMPS@9: (no value), con-amp-mt:L03P
- added U$10: (no value), Analog Devices - AD7997BRUZ-1REEL:AD7175
- added U$11, U$13, U$15, U$16, U$25, U$26, U$35: 100nF, Nordic_nRF:CAPACITOR_0603_N
- added U$12, U$42, U$45: 10uF, Nordic_nRF:CAPACITOR_0603_N
- added U$14, U$19, U$22, U$23, U$24, U$30, U$37, U$38, U$43, U$44, U$46, U$48: 0.1uF, Nordic_nRF:CAPACITOR_0603_N
- added U$17, U$18: TBD, Nordic_nRF:CAPACITOR_0603_N
- added U$20, U$31, U$47, U$49, U$71: 1uF, Nordic_nRF:CAPACITOR_0603_N
- added U$21: 4.7uF, Nordic_nRF:CAPACITOR_0603_N
- added U$33, U$34: 22nF, Nordic_nRF:CAPACITOR_0603_N
- added U$36: 10nF, Nordic_nRF:CAPACITOR_0603_N
- added U$70: PCF8575C, pcf8575c:PCF8575C
- added Y1: 16MHz, SparkFun-Clocks:CRYSTAL-26MHZSMD-3.2X2.5
- R14: value (none) -> 2k2; device adafruit:FLIPFLOP-RES -> SparkFun-Resistors:0.11OHM-2010-1/2W-1%
- R15: value (none) -> 3k3; device adafruit:FLIPFLOP-RES -> SparkFun-Resistors:0.11OHM-2010-1/2W-1%
- R17, R21, R25, R27: value (none) -> 10k; device adafruit:FLIPFLOP-RES -> SparkFun-Resistors:100KOHM-0603-1/10W-1%
- R18, R19, R20, R22, R24, R26, R28: value (none) -> 100k; device adafruit:FLIPFLOP-RES -> SparkFun-Resistors:100KOHM-0603-1/10W-1%
- U11: value (none) -> LTC6655CHMS8-3.3PBF; device SOP65P640X120-17N:BUCK_CONVERTER1 -> LTC6655CHMS8-3.3PBF:LTC6655CHMS8-3.3PBF
Connections:
- removed net N$41: U$6.18_SDA/SPI_CS_N
- removed net N$49: ENCODER@Y-4.S
- removed net SS: BUCKCONVERTER1.SS, C34.1
- new net ACC-INT: U1.INT, X1.GPIO17
- new net AGND: FB4.1, R18.1, R19.1, TEMPS@1-1.S, TEMPS@10-1.S, TEMPS@11-1.S, TEMPS@12-1.S, TEMPS@13-1.S, TEMPS@14-1.S, TEMPS@15-1.S, TEMPS@16-1.S, TEMPS@2-1.S, TEMPS@3-1.S, TEMPS@4-1.S, TEMPS@5-1.S, TEMPS@6-1.S, TEMPS@7-1.S, TEMPS@8-1.S, TEMPS@9-1.S, U$37.2, U$42.2, U$43.2, U$44.2, U$45.2, U$46.2, U$47.2, U$48.2, U$49.2, U6.1_AGND, U6.2_AGND, U6.3_AGND, U6.4_AGND, U8.1_AGND, U8.2_AGND, U8.3_AGND, U8.4_AGND, U8.AS
- new net BUCK-PG: X1.GPIO23
- new net CE2: ENCODER@Y-4.S, X1.GPIO05
- new net CE3: ENCODER@Z-4.S, X1.GPIO06
- new net CE4: X1.GPIO24
- new net CE5: X1.GPIO25
- new net CE6: X1.GPIO04
- new net COMP-INT: U7.INT, X1.GPIO27
- new net COMP-INT-TRIG: U7.INT/TRIG, X1.GPIO22
- new net GND: FB2.1, U$10.AVSS, U$10.REF-, U$11.2, U$12.2, U$13.2, U$14.2, U$15.2, U$19.2, U$20.2, U$21.2, U$22.2, U$23.1, U$24.1, U$26.2, U$35.2, U11.GND, U11.GND_2, U11.GND_3, U11.GND_4, U5B.1_AGND, U5B.2_AGND
- new net GPS-INT: U$6.4_EXTINT, X1.GPIO13
- new net GPS-LNA: U$6.14_LNA_EN/RESERVED, X1.GPIO19
- new net GPS-RESET: U$6.8_RESET_N, X1.GPIO12
- new net IO-INT: U$70.!INT, X1.GPIO18
- new net MOTOR-EN1: IC1.ENABLE_A, X1.GPIO16
- new net MOTOR-EN2: IC1.ENABLE_B, X1.GPIO26
- new net MOTOR-EN3: IC2.ENABLE_A, X1.GPIO20
- new net MOTOR-EN4: IC2.ENABLE_B, X1.GPIO21
- new net N$51: U$10.REFCAPD, U$30.1, U$31.1
- new net N$55: U$34.1, U5A.1_CP3, U5A.2_CP3
- new net N$60: U$46.1, U$47.1, U8.REFIN
- new net N$66: R37.1, U$10.GPIO0
- new net N$69: T1.C, TEMPA@1-2.S
- new net N$70: R20.1, R21.2, T2.B
- new net N$71: T2.C, TEMPA@2-2.S
- new net N$73: R22.1, R23.2, T3.B
- new net N$74: T3.C, TEMPA@3-2.S
- new net N$76: R24.1, R25.2, T4.B
- new net N$77: T4.C, TEMPA@4-2.S
- new net N$79: R26.1, R27.2, T5.B
- new net N$80: T5.C, TEMPA@5-2.S
- new net N$82: R28.1, R29.2, T6.B
- new net N$83: T6.C, TEMPA@6-2.S
- new net N$85: R30.1, R31.2, T7.B
- new net N$86: T7.C, TEMPA@7-2.S
- new net N$88: R32.1, R33.2, T8.B
- new net N$89: T8.C, TEMPA@8-2.S
- new net N$91: R34.1, R35.2, T9.B
- new net N$92: T9.C, TEMPA@9-2.S
- new net PWM-EN: U$70.P00, U4.!OE
- new net SDF: R36.2, U$10.DOUT/RDY
- new net TEMPA1: R17.1, U$70.P03
- new net TEMPA2: R21.1, U$70.P04
- new net TEMPA3: R23.1, U$70.P05
- new net TEMPA4: R25.1, U$70.P06
- new net TEMPA5: R27.1, U$70.P07
- new net TEMPA6: R29.1, U$70.P10
- new net TEMPA7: R31.1, U$70.P11
- new net TEMPA8: R33.1, U$70.P12
- new net TEMPA9: R35.1, U$70.P13
- new net TEMPS-INT1: U$70.P01
- new net TEMPS-INT2: U$70.P02
- new net TEMPS1: TEMPS@1-2.S, U6.VIN1
- new net TEMPS10: TEMPS@10-2.S, U8.VIN2
- new net TEMPS11: TEMPS@11-2.S, U8.VIN3
- new net TEMPS12: TEMPS@12-2.S, U8.VIN4
- new net TEMPS13: TEMPS@13-2.S, U8.VIN5
- new net TEMPS14: TEMPS@14-2.S, U8.VIN6
- new net TEMPS15: TEMPS@15-2.S, U8.VIN7
- new net TEMPS16: TEMPS@16-2.S, U8.VIN8
- new net TEMPS2: TEMPS@2-2.S, U6.VIN2
- new net TEMPS3: TEMPS@3-2.S, U6.VIN3
- new net TEMPS4: TEMPS@4-2.S, U6.VIN4
- new net TEMPS5: TEMPS@5-2.S, U6.VIN5
- new net TEMPS6: TEMPS@6-2.S, U6.VIN6
- new net TEMPS7: TEMPS@7-2.S, U6.VIN7
- new net TEMPS8: TEMPS@8-2.S, U6.VIN8
- new net TEMPS9: TEMPS@9-2.S, U8.VIN1
- new net VCCA: FB1.2, R38.1, U$10.AVDD1, U$10.AVDD2, U$11.1, U$15.1, U$23.2, U$24.2, U$26.1, U11.VIN, U11.~SHDN, U5B.1_AVCC, U5B.2_AVCC
- new net VCC_1: FB3.2, TEMPS@1-3.S, TEMPS@10-3.S, TEMPS@11-3.S, TEMPS@12-3.S, TEMPS@13-3.S, TEMPS@14-3.S, TEMPS@15-3.S, TEMPS@16-3.S, TEMPS@2-3.S, TEMPS@3-3.S, TEMPS@4-3.S, TEMPS@5-3.S, TEMPS@6-3.S, TEMPS@7-3.S, TEMPS@8-3.S, TEMPS@9-3.S, U$37.1, U$42.1, U$43.1, U$44.1, U$45.1, U6.1_VDD, U6.2_VDD, U6.AS, U8.1_VDD, U8.2_VDD
- net 0: now also FB2.2, FB4.2, R15.1, TEMPA@1-1.S, TEMPA@2-1.S, TEMPA@3-1.S, TEMPA@4-1.S, TEMPA@5-1.S, TEMPA@6-1.S, TEMPA@7-1.S, TEMPA@8-1.S, TEMPA@9-1.S, U$10.DGND, U$16.2, U$17.2, U$18.1, U$25.2, U$30.2, U$31.2, U$38.2, U$70.VSS, U$71.2, U1.ADDR, U4.A0, U4.A4, U5B.1_PGND, U5B.2_PGND, U7.A0, U7.A1, Y1.3; no longer BUCKCONVERTER1.GND, BUCK_CONVERTER2.FB, BUCK_CONVERTER2.SGND, C20.1, C21.1, C22.1, C23.1, C25.1, C26.1, C27.1, C29.1, C31.1, C32.1, C34.2, C35.1, C37.1, C38.1, C39.1, C40.1, C41.1, C42.1, C43.1, C44.1, R17.1, R19.1, R20.1, R22.1, R24.2, R26.2, R27.2, U11.AGND, U11.PGND1, U11.PGND2, U11.SYNC, U4.!OE
- net 12V: no longer C25.2, C43.2, C44.2, L4.2, R15.2
- net 3.3V: now also U$70.A0, U$70.A1, U$70.A2, U$70.VDD, U$71.1, U7.SENB/CS; no longer C29.2, C30.2, C32.2, C40.2, C41.2, L5.2, R21.2, R28.1, U11.BIAS
- net 5V: now also FB1.1, FB3.1, R14.2, R16.2, R20.2, R22.2, R24.2, R26.2, R28.2, R30.2, R32.2, R34.2, T1.E, T2.E, T3.E, T4.E, T5.E, T6.E, T7.E, T8.E, T9.E, U$16.1, U$25.1, U$38.1, U4.A1, U4.A2, U4.A3, U5B.1_VDD, U5B.2_VDD; no longer C37.2, C38.2, C39.2, L6.2, R25.1
- net CE0: now also U$6.18_SDA/SPI_CS_N
- net CE1: now also ENCODER@X-4.S
- net CLK: now also U$10.SCLK
- net MISO: now also R36.1
- net MOSI: now also U$10.DIN
- net N$40: now also U$10.XTAL1, U$17.1, Y1.1; no longer BUCK_CONVERTER2.RTN, R15.1, R17.2
- net N$42: now also SELF-TEST-1.S, U5A.1_ST1, U5A.2_ST1; no longer BUCK_CONVERTER2.VCC, C23.2
- net N$43: now also R38.2, T10.C; no longer ENCODER@Z-4.S
- net N$44: now also U$10.XTAL2, U$18.2, Y1.2; no longer BUCK_CONVERTER2.BST, C24.2
- net N$45: now also U$10.REGCAPA, U$19.1, U$20.1; no longer BUCK_CONVERTER2.SW, C24.1, D2.C, L4.1
- net N$46: now also R37.2, T10.B; no longer ENCODER@X-4.S
- net N$47: now also SELF-TEST-2.S, U5A.1_ST2, U5A.2_ST2; no longer BUCK_CONVERTER2.RON/SD, R14.1
- net N$48: now also U$10.REF+, U$12.1, U$13.1, U$14.1, U$21.1, U$22.1, U11.VOUT_F, U11.VOUT_S, U5B.1_VRATIO, U5B.2_VRATIO; no longer BUCK_CONVERTER2.SS, C22.2
- net N$50: now also R14.1, R15.2, U$10.IOVDD; no longer BUCK_CONVERTER2.ISEN, D2.A
- net N$52: now also U$35.1, U5A.1_CP5, U5A.2_CP5; no longer R18.1, R19.2, U11.EN
- net N$53: now also T10.E, U$36.2, U5A.1_SUMJ, U5A.2_SUMJ; no longer C27.2, U11.SS/TRK
- net N$54: now also U$34.2, U5A.1_CP4, U5A.2_CP4; no longer R20.2, U11.RT
- net N$56: now also U$33.2, U5A.1_CP2, U5A.2_CP2; no longer C28.2, L5.1, U11.SW1, U11.SW2
- net N$57: now also U$33.1, U5A.1_CP1, U5A.2_CP1; no longer C28.1, U11.CBOOT
- net N$58: now also U$10.AIN1, U$36.1, U5A.1_RATEOUT, U5A.2_RATEOUT; no longer C30.1, R21.1, R22.2, U11.FB
- net N$59: now also U$10.AIN0, U5A.1_TEMP, U5A.2_TEMP; no longer C31.2, U11.VCC
- net N$61: now also U$10.CS; no longer BUCKCONVERTER1.LX, C36.1, L6.1
- net N$62: now also R18.2, U8.ALERT/BUSY; no longer C33.1, R27.1
- net N$63: now also U$48.1, U$49.1, U6.REFIN; no longer BUCKCONVERTER1.FSW, R24.1
- net N$64: now also U8.!CONVST!; no longer BUCKCONVERTER1.COMP, C33.2
- net N$65: now also R16.1, R17.2, T1.B; no longer BUCKCONVERTER1.BST, C36.2
- net N$67: now also R19.2, U6.ALERT/BUSY; no longer BUCKCONVERTER1.FB, R25.2, R26.1
- net N$68: now also U6.!CONVST!; no longer R28.2, U11.PGOOD
- net SCL: now also U$70.SCL, U6.SCL, U8.SCL
- net SDA: now also U$70.SDA, U6.SDA, U8.SDA
- net VCC: no longer BUCKCONVERTER1.EN, BUCKCONVERTER1.VIN, BUCK_CONVERTER2.VIN, C20.2, C21.2, C26.2, C35.2, C42.2, R14.2, R18.2, U11.VIN1, U11.VIN2
Other:
- note added: "Thermal Actuators"
- note added: "Thermal Sensors"
- note removed: "Buck converter: AOZ1284PI"
- note removed: "Thermal"

Commit message: Revert "Merge branch 'master' into test"
This reverts commit dfcaf70d8e9cfdf546262c8a169c9a7cbb3319ac.
Parts:
- removed FB1, FB2, FB3, FB4: 30Ω/1.8A, SparkFun-Coils:FERRITE_BEAD-0603
- removed R16, R30, R32, R34, R38: 100k, SparkFun-Resistors:100KOHM-0603-1/10W-1%
- removed R23, R29, R31, R33, R35, R37: 10k, SparkFun-Resistors:100KOHM-0603-1/10W-1%
- removed R36: 5.6k, SparkFun-Resistors:5.6KOHM-0603-1/10W-1%
- removed SELF-TEST, TEMPA@1, TEMPA@2, TEMPA@3, TEMPA@4, TEMPA@5, TEMPA@6, TEMPA@7, TEMPA@8, TEMPA@9: (no value), con-amp-mt:L02P
- removed T1, T2, T3, T4, T5, T6, T7, T8, T9: (no value), DC_LOAD_AU:-PNP-SOT23-BEC
- removed T10: (no value), DC_LOAD_AU:-NPN-SOT23-BEC
- removed TEMPS@1, TEMPS@10, TEMPS@11, TEMPS@12, TEMPS@13, TEMPS@14, TEMPS@15, TEMPS@16, TEMPS@2, TEMPS@3, TEMPS@4, TEMPS@5, TEMPS@6, TEMPS@7, TEMPS@8, TEMPS@9: (no value), con-amp-mt:L03P
- removed U$10: (no value), Analog Devices - AD7997BRUZ-1REEL:AD7175
- removed U$11, U$13, U$15, U$16, U$25, U$26, U$35: 100nF, Nordic_nRF:CAPACITOR_0603_N
- removed U$12, U$42, U$45: 10uF, Nordic_nRF:CAPACITOR_0603_N
- removed U$14, U$19, U$22, U$23, U$24, U$30, U$37, U$38, U$43, U$44, U$46, U$48: 0.1uF, Nordic_nRF:CAPACITOR_0603_N
- removed U$17, U$18: TBD, Nordic_nRF:CAPACITOR_0603_N
- removed U$20, U$31, U$47, U$49, U$71: 1uF, Nordic_nRF:CAPACITOR_0603_N
- removed U$21: 4.7uF, Nordic_nRF:CAPACITOR_0603_N
- removed U$33, U$34: 22nF, Nordic_nRF:CAPACITOR_0603_N
- removed U$36: 10nF, Nordic_nRF:CAPACITOR_0603_N
- removed U$70: PCF8575C, pcf8575c:PCF8575C
- removed Y1: 16MHz, SparkFun-Clocks:CRYSTAL-26MHZSMD-3.2X2.5
- added BUCKCONVERTER1: (no value), SO-8:BUCK-CONVERTER5V4A
- added BUCK_CONVERTER2: LM2695MH, LM2695MH:LM2695MH
- added C20, C21: (no value), Wurth_Elektronik_Passive_Capacitors_rev18b:WCAP-CSGP_0805_885012006082_REFLOW
- added C22, C23, C24, C25, C26, C27, C28, C29, C30, C31, C32, C33, C34, C35, C36, C37, C38, C39, C40, C41, C42, C43, C44: (no value), Wurth_Elektronik_Passive_Capacitors_rev18b:WCAP-CSGP_0805_885012006018_WAVE
- added D2: (no value), BeagleBone_Blue_R3:DIODE
- added IC3, IC4, IC5: ADS1271, texas:ADS1271
- added L4, L5: (no value), BeagleBone_Blue_R3:INDUCTOR
- added L6: 22uH, BeagleBone_Blue_R3:INDUCTOR
- added SV1: (no value), con-amp-mt:L03P
- added U10, U9: ANALOG_DEVICES_ADXRS646BBGZANALOG_DEVICES_ADXRS646BBGZ_0_0, Analog Devices - ADXRS646BBGZ:ANALOG_DEVICES_ADXRS646BBGZANALOG_DEVICES_ADXRS646BBGZ_0_0
- R14: value 2k2 -> (none); device SparkFun-Resistors:0.11OHM-2010-1/2W-1% -> adafruit:FLIPFLOP-RES
- R15: value 3k3 -> (none); device SparkFun-Resistors:0.11OHM-2010-1/2W-1% -> adafruit:FLIPFLOP-RES
- R17, R21, R25, R27: value 10k -> (none); device SparkFun-Resistors:100KOHM-0603-1/10W-1% -> adafruit:FLIPFLOP-RES
- R18, R19, R20, R22, R24, R26, R28: value 100k -> (none); device SparkFun-Resistors:100KOHM-0603-1/10W-1% -> adafruit:FLIPFLOP-RES
- U11: value LTC6655CHMS8-3.3PBF -> (none); device LTC6655CHMS8-3.3PBF:LTC6655CHMS8-3.3PBF -> SOP65P640X120-17N:BUCK_CONVERTER1
Connections:
- removed net ACC-INT: U1.INT, X1.GPIO17
- removed net AGND: FB4.1, R18.1, R19.1, TEMPS@1-1.S, TEMPS@10-1.S, TEMPS@11-1.S, TEMPS@12-1.S, TEMPS@13-1.S, TEMPS@14-1.S, TEMPS@15-1.S, TEMPS@16-1.S, TEMPS@2-1.S, TEMPS@3-1.S, TEMPS@4-1.S, TEMPS@5-1.S, TEMPS@6-1.S, TEMPS@7-1.S, TEMPS@8-1.S, TEMPS@9-1.S, U$37.2, U$42.2, U$43.2, U$44.2, U$45.2, U$46.2, U$47.2, U$48.2, U$49.2, U6.1_AGND, U6.2_AGND, U6.3_AGND, U6.4_AGND, U8.1_AGND, U8.2_AGND, U8.3_AGND, U8.4_AGND, U8.AS
- removed net BUCK-PG: X1.GPIO23
- removed net CE2: ENCODER@Y-4.S, X1.GPIO05
- removed net CE3: ENCODER@Z-4.S, X1.GPIO06
- removed net CE4: X1.GPIO24
- removed net CE5: X1.GPIO25
- removed net CE6: X1.GPIO04
- removed net COMP-INT: U7.INT, X1.GPIO27
- removed net COMP-INT-TRIG: U7.INT/TRIG, X1.GPIO22
- removed net GND: FB2.1, U$10.AVSS, U$10.REF-, U$11.2, U$12.2, U$13.2, U$14.2, U$15.2, U$19.2, U$20.2, U$21.2, U$22.2, U$23.1, U$24.1, U$26.2, U$35.2, U11.GND, U11.GND_2, U11.GND_3, U11.GND_4, U5B.1_AGND, U5B.2_AGND
- removed net GPS-INT: U$6.4_EXTINT, X1.GPIO13
- removed net GPS-LNA: U$6.14_LNA_EN/RESERVED, X1.GPIO19
- removed net GPS-RESET: U$6.8_RESET_N, X1.GPIO12
- removed net IO-INT: U$70.!INT, X1.GPIO18
- removed net MOTOR-EN1: IC1.ENABLE_A, X1.GPIO16
- removed net MOTOR-EN2: IC1.ENABLE_B, X1.GPIO26
- removed net MOTOR-EN3: IC2.ENABLE_A, X1.GPIO20
- removed net MOTOR-EN4: IC2.ENABLE_B, X1.GPIO21
- removed net N$51: U$10.REFCAPD, U$30.1, U$31.1
- removed net N$55: U$34.1, U5A.1_CP3, U5A.2_CP3
- removed net N$60: U$46.1, U$47.1, U8.REFIN
- removed net N$66: R37.1, U$10.GPIO0
- removed net N$69: T1.C, TEMPA@1-2.S
- removed net N$70: R20.1, R21.2, T2.B
- removed net N$71: T2.C, TEMPA@2-2.S
- removed net N$73: R22.1, R23.2, T3.B
- removed net N$74: T3.C, TEMPA@3-2.S
- removed net N$76: R24.1, R25.2, T4.B
- removed net N$77: T4.C, TEMPA@4-2.S
- removed net N$79: R26.1, R27.2, T5.B
- removed net N$80: T5.C, TEMPA@5-2.S
- removed net N$82: R28.1, R29.2, T6.B
- removed net N$83: T6.C, TEMPA@6-2.S
- removed net N$85: R30.1, R31.2, T7.B
- removed net N$86: T7.C, TEMPA@7-2.S
- removed net N$88: R32.1, R33.2, T8.B
- removed net N$89: T8.C, TEMPA@8-2.S
- removed net N$91: R34.1, R35.2, T9.B
- removed net N$92: T9.C, TEMPA@9-2.S
- removed net PWM-EN: U$70.P00, U4.!OE
- removed net SDF: R36.2, U$10.DOUT/RDY
- removed net TEMPA1: R17.1, U$70.P03
- removed net TEMPA2: R21.1, U$70.P04
- removed net TEMPA3: R23.1, U$70.P05
- removed net TEMPA4: R25.1, U$70.P06
- removed net TEMPA5: R27.1, U$70.P07
- removed net TEMPA6: R29.1, U$70.P10
- removed net TEMPA7: R31.1, U$70.P11
- removed net TEMPA8: R33.1, U$70.P12
- removed net TEMPA9: R35.1, U$70.P13
- removed net TEMPS-INT1: U$70.P01
- removed net TEMPS-INT2: U$70.P02
- removed net TEMPS1: TEMPS@1-2.S, U6.VIN1
- removed net TEMPS10: TEMPS@10-2.S, U8.VIN2
- removed net TEMPS11: TEMPS@11-2.S, U8.VIN3
- removed net TEMPS12: TEMPS@12-2.S, U8.VIN4
- removed net TEMPS13: TEMPS@13-2.S, U8.VIN5
- removed net TEMPS14: TEMPS@14-2.S, U8.VIN6
- removed net TEMPS15: TEMPS@15-2.S, U8.VIN7
- removed net TEMPS16: TEMPS@16-2.S, U8.VIN8
- removed net TEMPS2: TEMPS@2-2.S, U6.VIN2
- removed net TEMPS3: TEMPS@3-2.S, U6.VIN3
- removed net TEMPS4: TEMPS@4-2.S, U6.VIN4
- removed net TEMPS5: TEMPS@5-2.S, U6.VIN5
- removed net TEMPS6: TEMPS@6-2.S, U6.VIN6
- removed net TEMPS7: TEMPS@7-2.S, U6.VIN7
- removed net TEMPS8: TEMPS@8-2.S, U6.VIN8
- removed net TEMPS9: TEMPS@9-2.S, U8.VIN1
- removed net VCCA: FB1.2, R38.1, U$10.AVDD1, U$10.AVDD2, U$11.1, U$15.1, U$23.2, U$24.2, U$26.1, U11.VIN, U11.~SHDN, U5B.1_AVCC, U5B.2_AVCC
- removed net VCC_1: FB3.2, TEMPS@1-3.S, TEMPS@10-3.S, TEMPS@11-3.S, TEMPS@12-3.S, TEMPS@13-3.S, TEMPS@14-3.S, TEMPS@15-3.S, TEMPS@16-3.S, TEMPS@2-3.S, TEMPS@3-3.S, TEMPS@4-3.S, TEMPS@5-3.S, TEMPS@6-3.S, TEMPS@7-3.S, TEMPS@8-3.S, TEMPS@9-3.S, U$37.1, U$42.1, U$43.1, U$44.1, U$45.1, U6.1_VDD, U6.2_VDD, U6.AS, U8.1_VDD, U8.2_VDD
- new net N$41: U$6.18_SDA/SPI_CS_N
- new net N$49: ENCODER@Y-4.S
- new net SS: BUCKCONVERTER1.SS, C34.1
- net 0: now also BUCKCONVERTER1.GND, BUCK_CONVERTER2.FB, BUCK_CONVERTER2.SGND, C20.1, C21.1, C22.1, C23.1, C25.1, C26.1, C27.1, C29.1, C31.1, C32.1, C34.2, C35.1, C37.1, C38.1, C39.1, C40.1, C41.1, C42.1, C43.1, C44.1, R17.1, R19.1, R20.1, R22.1, R24.2, R26.2, R27.2, U11.AGND, U11.PGND1, U11.PGND2, U11.SYNC, U4.!OE; no longer FB2.2, FB4.2, R15.1, TEMPA@1-1.S, TEMPA@2-1.S, TEMPA@3-1.S, TEMPA@4-1.S, TEMPA@5-1.S, TEMPA@6-1.S, TEMPA@7-1.S, TEMPA@8-1.S, TEMPA@9-1.S, U$10.DGND, U$16.2, U$17.2, U$18.1, U$25.2, U$30.2, U$31.2, U$38.2, U$70.VSS, U$71.2, U1.ADDR, U4.A0, U4.A4, U5B.1_PGND, U5B.2_PGND, U7.A0, U7.A1, Y1.3
- net 12V: now also C25.2, C43.2, C44.2, L4.2, R15.2
- net 3.3V: now also C29.2, C30.2, C32.2, C40.2, C41.2, L5.2, R21.2, R28.1, U11.BIAS; no longer U$70.A0, U$70.A1, U$70.A2, U$70.VDD, U$71.1, U7.SENB/CS
- net 5V: now also C37.2, C38.2, C39.2, L6.2, R25.1; no longer FB1.1, FB3.1, R14.2, R16.2, R20.2, R22.2, R24.2, R26.2, R28.2, R30.2, R32.2, R34.2, T1.E, T2.E, T3.E, T4.E, T5.E, T6.E, T7.E, T8.E, T9.E, U$16.1, U$25.1, U$38.1, U4.A1, U4.A2, U4.A3, U5B.1_VDD, U5B.2_VDD
- net CE0: no longer U$6.18_SDA/SPI_CS_N
- net CE1: no longer ENCODER@X-4.S
- net CLK: no longer U$10.SCLK
- net MISO: no longer R36.1
- net MOSI: no longer U$10.DIN
- net N$40: now also BUCK_CONVERTER2.RTN, R15.1, R17.2; no longer U$10.XTAL1, U$17.1, Y1.1
- net N$42: now also BUCK_CONVERTER2.VCC, C23.2; no longer SELF-TEST-1.S, U5A.1_ST1, U5A.2_ST1
- net N$43: now also ENCODER@Z-4.S; no longer R38.2, T10.C
- net N$44: now also BUCK_CONVERTER2.BST, C24.2; no longer U$10.XTAL2, U$18.2, Y1.2
- net N$45: now also BUCK_CONVERTER2.SW, C24.1, D2.C, L4.1; no longer U$10.REGCAPA, U$19.1, U$20.1
- net N$46: now also ENCODER@X-4.S; no longer R37.2, T10.B
- net N$47: now also BUCK_CONVERTER2.RON/SD, R14.1; no longer SELF-TEST-2.S, U5A.1_ST2, U5A.2_ST2
- net N$48: now also BUCK_CONVERTER2.SS, C22.2; no longer U$10.REF+, U$12.1, U$13.1, U$14.1, U$21.1, U$22.1, U11.VOUT_F, U11.VOUT_S, U5B.1_VRATIO, U5B.2_VRATIO
- net N$50: now also BUCK_CONVERTER2.ISEN, D2.A; no longer R14.1, R15.2, U$10.IOVDD
- net N$52: now also R18.1, R19.2, U11.EN; no longer U$35.1, U5A.1_CP5, U5A.2_CP5
- net N$53: now also C27.2, U11.SS/TRK; no longer T10.E, U$36.2, U5A.1_SUMJ, U5A.2_SUMJ
- net N$54: now also R20.2, U11.RT; no longer U$34.2, U5A.1_CP4, U5A.2_CP4
- net N$56: now also C28.2, L5.1, U11.SW1, U11.SW2; no longer U$33.2, U5A.1_CP2, U5A.2_CP2
- net N$57: now also C28.1, U11.CBOOT; no longer U$33.1, U5A.1_CP1, U5A.2_CP1
- net N$58: now also C30.1, R21.1, R22.2, U11.FB; no longer U$10.AIN1, U$36.1, U5A.1_RATEOUT, U5A.2_RATEOUT
- net N$59: now also C31.2, U11.VCC; no longer U$10.AIN0, U5A.1_TEMP, U5A.2_TEMP
- net N$61: now also BUCKCONVERTER1.LX, C36.1, L6.1; no longer U$10.CS
- net N$62: now also C33.1, R27.1; no longer R18.2, U8.ALERT/BUSY
- net N$63: now also BUCKCONVERTER1.FSW, R24.1; no longer U$48.1, U$49.1, U6.REFIN
- net N$64: now also BUCKCONVERTER1.COMP, C33.2; no longer U8.!CONVST!
- net N$65: now also BUCKCONVERTER1.BST, C36.2; no longer R16.1, R17.2, T1.B
- net N$67: now also BUCKCONVERTER1.FB, R25.2, R26.1; no longer R19.2, U6.ALERT/BUSY
- net N$68: now also R28.2, U11.PGOOD; no longer U6.!CONVST!
- net SCL: no longer U$70.SCL, U6.SCL, U8.SCL
- net SDA: no longer U$70.SDA, U6.SDA, U8.SDA
- net VCC: now also BUCKCONVERTER1.EN, BUCKCONVERTER1.VIN, BUCK_CONVERTER2.VIN, C20.2, C21.2, C26.2, C35.2, C42.2, R14.2, R18.2, U11.VIN1, U11.VIN2
Other:
- note added: "Buck converter: AOZ1284PI"
- note added: "Thermal"
- note removed: "Thermal Actuators"
- note removed: "Thermal Sensors"
