File: 1st iteration/E-Accelerometer/irisc.brd (EAGLE design)
At the start: 20.3 x 11.1 mm, 4 parts, among them U1 KXTJ3-1057

Commit message: E's systems almost done (only PCB gyro missing)
Parts:
- moved U$8 1.25 mm to (13.8, 6.86)
- moved J2 1.25 mm to (3.68, 3.05)
- moved U1 1.25 mm to (8.76, 5.59)
- moved J1 1.25 mm to (18.9, 5.59)
Routing:
- net 0: track 50.4 -> 49.8 mm
Other:
- board size 20.3 x 11.1 mm -> 21.4 x 11.6 mm
