File: 1st iteration/E-IO expender/irisc.brd (EAGLE design)
At the start: 40.5 x 34.5 mm, 6 parts

Commit message: E's systems almost done (only PCB gyro missing)
Routing:
- net 0: track 7.14 -> 64.4 mm
- removed copper zone on layer 1, net 0
