File: 1st iteration/E-Motorcontroller/irisc.brd (EAGLE design)
At the start: 76.2 x 50.5 mm, 17 parts, among them IC1 L298, U4 PCA9685

Commit message: E's systems almost done (only PCB gyro missing)
Parts:
- removed J2: (no value), SparkFun-Connectors:1X05
- removed U$5: 1uF, Nordic_nRF:RESC0805_L
- removed U4: PCA9685, SparkFun-IC-Special-Function:TSSOP-28_4MM
- added J5: (no value), SparkFun-Connectors:1X02
- added J6: (no value), SparkFun-Connectors:1X03
- added U$1: 1uF, Nordic_nRF:RESC0805_L
- added U1: PCA9685, SparkFun-IC-Special-Function:TSSOP-28_4MM
- moved J1 19.7 mm to (14.2, 10.8)
- moved U$4 13.8 mm to (23.1, 26.0), turned to 90 degrees
- moved U$3 12.0 mm to (21.4, 18.9)
- moved IC1 4.02 mm to (26.7, 25.4)
Connections:
- net 0: now also U$1.2, U1.1, U1.14, U1.24, U1.25, U1.5; no longer U$5.2, U4.1, U4.14, U4.24, U4.25, U4.5
- net 5V: now also U$1.1, U1.2, U1.28, U1.3, U1.4; no longer U$5.1, U4.2, U4.28, U4.3, U4.4
- net MOTOR-EN1: now also J5.2; no longer J2.2
- net MOTOR-EN2: now also J5.1; no longer J2.1
- net N$1: now also U1.19; no longer U4.22
- net N$10: now also U1.21; no longer U4.20
- net N$19: now also U1.22; no longer U4.19
- net N$5: now also U1.20; no longer U4.21
- net PWM_EN: now also J6.1, U1.23; no longer J2.3, U4.23
- net SCL: now also J6.2, U1.26; no longer J2.4, U4.26
- net SDA: now also J6.3, U1.27; no longer J2.5, U4.27
Routing:
- net 0: track 0.00 -> 193.5 mm, vias 0 -> 7
- net 12V: track 0.00 -> 137.6 mm, vias 0 -> 2
- net 5V: track 0.00 -> 58.3 mm, vias 0 -> 2
- net N$31: track 0.00 -> 45.3 mm
- net N$34: track 0.00 -> 43.8 mm
- net N$32: track 0.00 -> 41.4 mm
- net N$33: track 0.00 -> 38.6 mm
- net N$1: track 0.00 -> 25.7 mm
- net N$5: track 0.00 -> 24.9 mm
- net N$19: track 0.00 -> 18.9 mm
- net N$10: track 0.00 -> 18.5 mm
- net PWM_EN: track 0.00 -> 17.1 mm
- net MOTOR-EN1: track 0.00 -> 16.7 mm
- net SCL: track 0.00 -> 14.6 mm
- net SDA: track 0.00 -> 12.7 mm
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- added copper zone on layer 1, net 0
