File: 1st iteration/E-Gyroscopes/irisc.sch (EAGLE design)
At the start: 173 parts, among them IC1 L298, IC2 L298, U1 KXTJ3-1057, U11 LTC6655CHMS8-3.3PBF, U4 PCA9685, U5 ANALOG_DEVICES_ADXRS646BBGZAN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, U6 ANALOG_DEVICES_AD7997BRUZ-1RE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, U7 MELEXIS_TECHNOLOGIES_MLX90393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, U8 ANALOG_DEVICES_AD7997BRUZ-1RE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, X1 RASPI_BOARD_B+_E4, Y1 16MHz

Commit message: Removed unnecessary stuff in Elrick's 1st iteration PCB's
Parts:
- removed BUCKCONVERTER1: (no value), SO-8:BUCK-CONVERTER5V4A
- removed BUCK_CONVERTER3: LM2695MH, LM2695MH:LM2695MH
- removed C39: 0.1 uF, Wurth_Elektronik_Passive_Capacitors_rev18b:WCAP-CSGP_0805_885012006082_REFLOW
- removed C40: 3 uF, Wurth_Elektronik_Passive_Capacitors_rev18b:WCAP-CSGP_0805_885012006082_REFLOW
- removed C41: 492 nF, Wurth_Elektronik_Passive_Capacitors_rev18b:WCAP-CSGP_0805_885012006018_WAVE
- removed C42, C51: 1 uF, Wurth_Elektronik_Passive_Capacitors_rev18b:WCAP-CSGP_0805_885012006018_WAVE
- removed C43: 22 pF, Wurth_Elektronik_Passive_Capacitors_rev18b:WCAP-CSGP_0805_885012006018_WAVE
- removed C44, C62, C63: 4 uF, Wurth_Elektronik_Passive_Capacitors_rev18b:WCAP-CSGP_0805_885012006018_WAVE
- removed C45: 10 uF, Wurth_Elektronik_Passive_Capacitors_rev18b:WCAP-CSGP_0805_885012006018_WAVE
- removed C46: 22pF, Wurth_Elektronik_Passive_Capacitors_rev18b:WCAP-CSGP_0805_885012006018_WAVE
- removed C47: 47 uF, Wurth_Elektronik_Passive_Capacitors_rev18b:WCAP-CSGP_0805_885012006018_WAVE
- removed C48, C59, C60: 220 uF, Wurth_Elektronik_Passive_Capacitors_rev18b:WCAP-CSGP_0805_885012006018_WAVE
- removed C49: 44 pF, Wurth_Elektronik_Passive_Capacitors_rev18b:WCAP-CSGP_0805_885012006018_WAVE
- removed C50: 2.2 uF, Wurth_Elektronik_Passive_Capacitors_rev18b:WCAP-CSGP_0805_885012006018_WAVE
- removed C52: 100 nF, Wurth_Elektronik_Passive_Capacitors_rev18b:WCAP-CSGP_0805_885012006018_WAVE
- removed C53, C57, C58: 32 uF, Wurth_Elektronik_Passive_Capacitors_rev18b:WCAP-CSGP_0805_885012006018_WAVE
- removed C54: 1.44 pF, Wurth_Elektronik_Passive_Capacitors_rev18b:WCAP-CSGP_0805_885012006018_WAVE
- removed C55: 850 pF, Wurth_Elektronik_Passive_Capacitors_rev18b:WCAP-CSGP_0805_885012006018_WAVE
- removed C56: 3 uF, Wurth_Elektronik_Passive_Capacitors_rev18b:WCAP-CSGP_0805_885012006018_WAVE
- removed C61: 0.1 uF, Wurth_Elektronik_Passive_Capacitors_rev18b:WCAP-CSGP_0805_885012006018_WAVE
- removed D3: 0.75, BeagleBone_Blue_R3:DIODE
- removed ENCODER@X, ENCODER@Y, ENCODER@Z: (no value), con-amp-mt:L05P
- removed FB3, FB4: 30Ω/1.8A, SparkFun-Coils:FERRITE_BEAD-0603
- removed IC1, IC2: L298, st-microelectronics:L298
- removed J1: (no value), Wurth_Elektronik_Electromechanic_Coaxial _Connectors_rev18a:60314202124525
- removed L7: 24 uH, BeagleBone_Blue_R3:INDUCTOR
- removed L8: 68 uH, BeagleBone_Blue_R3:INDUCTOR
- removed L9: 22uH, BeagleBone_Blue_R3:INDUCTOR
- removed MOTOR@R, MOTOR@X, MOTOR@Y, MOTOR@Z, TEMPA@1, TEMPA@2, TEMPA@3, TEMPA@4, TEMPA@5, TEMPA@6, TEMPA@7, TEMPA@8, TEMPA@9: (no value), con-amp-mt:L02P
- removed R16, R18, R19, R20, R22, R24, R26, R28, R30, R32, R34: 100k, SparkFun-Resistors:100KOHM-0603-1/10W-1%
- removed R17, R21, R23, R25, R27, R29, R31, R33, R35: 10k, SparkFun-Resistors:100KOHM-0603-1/10W-1%
- removed R52: 470 k, adafruit:FLIPFLOP-RES
- removed R53: 47 k, adafruit:FLIPFLOP-RES
- removed R54: 12 k, adafruit:FLIPFLOP-RES
- removed R55, R56, R58: 1 M, adafruit:FLIPFLOP-RES
- removed R57: 200 k, adafruit:FLIPFLOP-RES
- removed R59: 442 k, adafruit:FLIPFLOP-RES
- removed R60: 56 k, adafruit:FLIPFLOP-RES
- removed R61, R64: 10 k, adafruit:FLIPFLOP-RES
- removed R62: 270 k, adafruit:FLIPFLOP-RES
- removed R63: 27 k, adafruit:FLIPFLOP-RES
- removed T1, T2, T3, T4, T5, T6, T7, T8, T9: (no value), DC_LOAD_AU:-PNP-SOT23-BEC
- removed TEMPS@1, TEMPS@10, TEMPS@11, TEMPS@12, TEMPS@13, TEMPS@14, TEMPS@15, TEMPS@16, TEMPS@2, TEMPS@3, TEMPS@4, TEMPS@5, TEMPS@6, TEMPS@7, TEMPS@8, TEMPS@9: (no value), con-amp-mt:L03P
- removed U$1, U$2, U$3, U$4: 100nF, Nordic_nRF:CAPACITOR_0805_L
- removed U$37, U$38, U$43, U$44, U$46, U$48: 0.1uF, Nordic_nRF:CAPACITOR_0603_N
- removed U$42, U$45: 10uF, Nordic_nRF:CAPACITOR_0603_N
- removed U$47, U$49, U$7, U$71, U$8, U$9: 1uF, Nordic_nRF:CAPACITOR_0603_N
- removed U$5: 1uF, Nordic_nRF:CAPACITOR_0805_L
- removed U$6: NEO-M8, ubloxLib:NEO-M8
- removed U$70: PCF8575C, pcf8575c:PCF8575C
- removed U1: KXTJ3-1057, KXTJ3-1057:KXTJ3-1057
- removed U20: (no value), SOP65P640X120-17N:BUCK_CONVERTER1
- removed U4: PCA9685, SparkFun-IC-Special-Function:PCA9685
- removed U6, U8: ANALOG_DEVICES_AD7997BRUZ-1REELANALOG_DEVICES_AD7997BRUZ-1R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, Analog Devices - AD7997BRUZ-1REEL:ANALOG_DEVICES_AD7997BRUZ-1REELANALOG_DEVICES_AD7997BRUZ-1REEL_0_0
- removed U7: MELEXIS_TECHNOLOGIES_MLX90393SLW-ABA-011-REMELEXIS_TECHNOLO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, Melexis Technologies - MLX90393SLW-ABA-011-RE:MELEXIS_TECHNOLOGIES_MLX90393SLW-ABA-011-REMELEXIS_TECHNOLOGIES_MLX90393S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
- removed X1: RASPI_BOARD_B+_E4, raspberrypi_bastelstube_v13:RASPI_BOARD_B+_E4
Connections:
- removed net 12V: C44.2, C62.2, C63.2, IC1.VS, IC2.VS, L7.2, R53.2, U$1.1, U$3.1
- removed net 3.3V: C48.2, C49.2, C51.2, C59.2, C60.2, L8.2, R58.2, R64.1, U$6.23_VCC, U$7.2, U$70.A0, U$70.A1, U$70.A2, U$70.VDD, U$71.1, U$8.1, U$9.1, U1.IO_VDD, U1.VDD, U20.BIAS, U7.SENB/CS, U7.VDD, U7.VDD_IO
- removed net ACC-INT: U1.INT, X1.GPIO17
- removed net AGND: FB4.1, R18.1, R19.1, TEMPS@1-1.S, TEMPS@10-1.S, TEMPS@11-1.S, TEMPS@12-1.S, TEMPS@13-1.S, TEMPS@14-1.S, TEMPS@15-1.S, TEMPS@16-1.S, TEMPS@2-1.S, TEMPS@3-1.S, TEMPS@4-1.S, TEMPS@5-1.S, TEMPS@6-1.S, TEMPS@7-1.S, TEMPS@8-1.S, TEMPS@9-1.S, U$37.2, U$42.2, U$43.2, U$44.2, U$45.2, U$46.2, U$47.2, U$48.2, U$49.2, U6.1_AGND, U6.2_AGND, U6.3_AGND, U6.4_AGND, U8.1_AGND, U8.2_AGND, U8.3_AGND, U8.4_AGND, U8.AS
- removed net BUCK-PG: X1.GPIO23
- removed net CE0: U$6.18_SDA/SPI_CS_N, X1.SPI_CE0
- removed net CE1: ENCODER@X-4.S, X1.SPI_CE1
- removed net CE2: ENCODER@Y-4.S, X1.GPIO05
- removed net CE3: ENCODER@Z-4.S, X1.GPIO06
- removed net CE4: X1.GPIO24
- removed net CE5: X1.GPIO25
- removed net CE6: X1.GPIO04
- removed net COMP-INT: U7.INT, X1.GPIO27
- removed net COMP-INT-TRIG: U7.INT/TRIG, X1.GPIO22
- removed net GPS-INT: U$6.4_EXTINT, X1.GPIO13
- removed net GPS-LNA: U$6.14_LNA_EN/RESERVED, X1.GPIO19
- removed net GPS-RESET: U$6.8_RESET_N, X1.GPIO12
- removed net IO-INT: U$70.!INT, X1.GPIO18
- removed net MOTOR-EN1: IC1.ENABLE_A, X1.GPIO16
- removed net MOTOR-EN2: IC1.ENABLE_B, X1.GPIO26
- removed net MOTOR-EN3: IC2.ENABLE_A, X1.GPIO20
- removed net MOTOR-EN4: IC2.ENABLE_B, X1.GPIO21
- removed net N$1: IC1.INPUT1, U4.CH15
- removed net N$10: IC1.INPUT3, U4.CH13
- removed net N$123: BUCK_CONVERTER3.RTN, R53.1, R54.2
- removed net N$124: BUCK_CONVERTER3.VCC, C42.2
- removed net N$125: BUCK_CONVERTER3.BST, C43.2
- removed net N$126: BUCK_CONVERTER3.SW, C43.1, D3.C, L7.1
- removed net N$127: BUCK_CONVERTER3.RON/SD, R52.1
- removed net N$128: BUCK_CONVERTER3.SS, C41.2
- removed net N$129: BUCK_CONVERTER3.ISEN, D3.A
- removed net N$130: R55.1, R56.2, U20.EN
- removed net N$131: C46.2, U20.SS/TRK
- removed net N$132: C47.2, L8.1, U20.SW1, U20.SW2
- removed net N$133: C47.1, U20.CBOOT
- removed net N$134: C49.1, R58.1, R59.2, U20.FB
- removed net N$135: C50.2, U20.VCC
- removed net N$136: BUCKCONVERTER1.LX, C52.1, L9.1
- removed net N$137: BUCKCONVERTER1.FSW, R62.1
- removed net N$138: BUCKCONVERTER1.COMP, C54.2
- removed net N$139: BUCKCONVERTER1.BST, C52.2
- removed net N$140: BUCKCONVERTER1.FB, R60.2, R61.1
- removed net N$141: C54.1, R63.1
- removed net N$142: R64.2, U20.PGOOD
- removed net N$143: R57.2, U20.RT
- removed net N$19: IC1.INPUT4, U4.CH12
- removed net N$22: IC2.INPUT1, U4.CH11
- removed net N$27: IC2.INPUT2, U4.CH10
- removed net N$28: IC2.INPUT3, U4.CH9
- removed net N$30: IC2.INPUT4, U4.CH8
- removed net N$31: IC1.OUT1, MOTOR@X-1.S
- removed net N$32: IC1.OUT2, MOTOR@X-2.S
- removed net N$33: IC1.OUT3, MOTOR@Y-1.S
- removed net N$34: IC1.OUT4, MOTOR@Y-2.S
- removed net N$35: IC2.OUT1, MOTOR@Z-1.S
- removed net N$36: IC2.OUT2, MOTOR@Z-2.S
- removed net N$37: IC2.OUT3, MOTOR@R-1.S
- removed net N$38: IC2.OUT4, MOTOR@R-2.S
- removed net N$39: J1.1, U$6.11_RF_IN
- removed net N$5: IC1.INPUT2, U4.CH14
- removed net N$60: U$46.1, U$47.1, U8.REFIN
- removed net N$62: R18.2, U8.ALERT/BUSY
- removed net N$63: U$48.1, U$49.1, U6.REFIN
- removed net N$64: U8.!CONVST!
- removed net N$65: R16.1, R17.2, T1.B
- removed net N$67: R19.2, U6.ALERT/BUSY
- removed net N$68: U6.!CONVST!
- removed net N$69: T1.C, TEMPA@1-2.S
- removed net N$70: R20.1, R21.2, T2.B
- removed net N$71: T2.C, TEMPA@2-2.S
- removed net N$73: R22.1, R23.2, T3.B
- removed net N$74: T3.C, TEMPA@3-2.S
- removed net N$76: R24.1, R25.2, T4.B
- removed net N$77: T4.C, TEMPA@4-2.S
- removed net N$79: R26.1, R27.2, T5.B
- removed net N$80: T5.C, TEMPA@5-2.S
- removed net N$82: R28.1, R29.2, T6.B
- removed net N$83: T6.C, TEMPA@6-2.S
- removed net N$85: R30.1, R31.2, T7.B
- removed net N$86: T7.C, TEMPA@7-2.S
- removed net N$88: R32.1, R33.2, T8.B
- removed net N$89: T8.C, TEMPA@8-2.S
- removed net N$91: R34.1, R35.2, T9.B
- removed net N$92: T9.C, TEMPA@9-2.S
- removed net PWM-EN: U$70.P00, U4.!OE
- removed net SCL: U$70.SCL, U1.SCL, U4.SCL, U6.SCL, U7.SCL/SCLK, U8.SCL, X1.SCL
- removed net SDA: U$70.SDA, U1.SDA, U4.SDA, U6.SDA, U7.SDA/MOSI, U8.SDA, X1.SDA
- removed net SS: BUCKCONVERTER1.SS, C55.1
- removed net SYNC: C46.1, R56.1, R57.1, U20.AGND, U20.SYNC
- removed net TEMPA1: R17.1, U$70.P03
- removed net TEMPA2: R21.1, U$70.P04
- removed net TEMPA3: R23.1, U$70.P05
- removed net TEMPA4: R25.1, U$70.P06
- removed net TEMPA5: R27.1, U$70.P07
- removed net TEMPA6: R29.1, U$70.P10
- removed net TEMPA7: R31.1, U$70.P11
- removed net TEMPA8: R33.1, U$70.P12
- removed net TEMPA9: R35.1, U$70.P13
- removed net TEMPS-INT1: U$70.P01
- removed net TEMPS-INT2: U$70.P02
- removed net TEMPS1: TEMPS@1-2.S, U6.VIN1
- removed net TEMPS10: TEMPS@10-2.S, U8.VIN2
- removed net TEMPS11: TEMPS@11-2.S, U8.VIN3
- removed net TEMPS12: TEMPS@12-2.S, U8.VIN4
- removed net TEMPS13: TEMPS@13-2.S, U8.VIN5
- removed net TEMPS14: TEMPS@14-2.S, U8.VIN6
- removed net TEMPS15: TEMPS@15-2.S, U8.VIN7
- removed net TEMPS16: TEMPS@16-2.S, U8.VIN8
- removed net TEMPS2: TEMPS@2-2.S, U6.VIN2
- removed net TEMPS3: TEMPS@3-2.S, U6.VIN3
- removed net TEMPS4: TEMPS@4-2.S, U6.VIN4
- removed net TEMPS5: TEMPS@5-2.S, U6.VIN5
- removed net TEMPS6: TEMPS@6-2.S, U6.VIN6
- removed net TEMPS7: TEMPS@7-2.S, U6.VIN7
- removed net TEMPS8: TEMPS@8-2.S, U6.VIN8
- removed net TEMPS9: TEMPS@9-2.S, U8.VIN1
- removed net VCC: BUCKCONVERTER1.EN, BUCKCONVERTER1.VIN, BUCK_CONVERTER3.VIN, C39.2, C40.2, C45.2, C56.2, C61.2, R52.2, R55.2, U20.VIN1, U20.VIN2
- removed net VCC_1: FB3.2, TEMPS@1-3.S, TEMPS@10-3.S, TEMPS@11-3.S, TEMPS@12-3.S, TEMPS@13-3.S, TEMPS@14-3.S, TEMPS@15-3.S, TEMPS@16-3.S, TEMPS@2-3.S, TEMPS@3-3.S, TEMPS@4-3.S, TEMPS@5-3.S, TEMPS@6-3.S, TEMPS@7-3.S, TEMPS@8-3.S, TEMPS@9-3.S, U$37.1, U$42.1, U$43.1, U$44.1, U$45.1, U6.1_VDD, U6.2_VDD, U6.AS, U8.1_VDD, U8.2_VDD
- net 0: no longer BUCK_CONVERTER3.FB, BUCK_CONVERTER3.SGND, C39.1, C40.1, C41.1, C42.1, C44.1, C45.1, C48.1, C50.1, C51.1, C53.1, C55.2, C56.1, C57.1, C58.1, C59.1, C60.1, C61.1, C62.1, C63.1, ENCODER@X-5.S, ENCODER@Y-5.S, ENCODER@Z-5.S, FB4.2, IC1.GND, IC1.SEN_A, IC1.SEN_B, IC2.GND, IC2.SEN_A, IC2.SEN_B, J1.2, R54.1, R59.1, R61.2, R62.2, R63.2, TEMPA@1-1.S, TEMPA@2-1.S, TEMPA@3-1.S, TEMPA@4-1.S, TEMPA@5-1.S, TEMPA@6-1.S, TEMPA@7-1.S, TEMPA@8-1.S, TEMPA@9-1.S, U$1.2, U$2.1, U$3.2, U$38.2, U$4.1, U$5.2, U$6.10_GND, U$6.12_GND, U$6.13_GND, U$6.24_GND, U$6.2_D_SEL, U$7.1, U$70.VSS, U$71.2, U$8.2, U$9.2, U1.ADDR, U1.GND, U1.RES, U20.PGND1, U20.PGND2, U4.A0, U4.A4, U4.A5, U4.EXTCLK, U4.VSS, U7.A0, U7.A1, U7.GND_PAD, U7.VSS, X1.GND
- net 5V: no longer C53.2, C57.2, C58.2, ENCODER@X-1.S, ENCODER@Y-1.S, ENCODER@Z-1.S, FB3.1, IC1.VCC, IC2.VCC, L9.2, R16.2, R20.2, R22.2, R24.2, R26.2, R28.2, R30.2, R32.2, R34.2, R60.1, T1.E, T2.E, T3.E, T4.E, T5.E, T6.E, T7.E, T8.E, T9.E, U$2.2, U$38.1, U$4.2, U$5.1, U4.A1, U4.A2, U4.A3, U4.VDD, X1.5V0
- net CLK: no longer ENCODER@X-3.S, ENCODER@Y-3.S, ENCODER@Z-3.S, U$6.19_SCL/SPI_CLK, X1.SPI_SCLK
- net GND: no longer BUCKCONVERTER1.GND
- net MISO: no longer ENCODER@X-2.S, ENCODER@Y-2.S, ENCODER@Z-2.S, U$6.20_TXD/SPI_MISO, X1.SPI_MISO
- net MOSI: no longer U$6.21_RXD/SPI_MOSI, X1.SPI_MOSI
Other:
- note removed: "Buck converter: AOZ1284PI"
- note removed: "Buck converter: LM2695MH"
- note removed: "Buck converter: LM43600PWPR"
- note removed: "Motor controller"
- note removed: "Power Management"
- note removed: "Sensors and onboard computer"
- note removed: "Thermal Actuators"
- note removed: "Thermal Sensors"

Commit message: 1st iteration update, beginning of the PCB's
Parts:
- added SV1: (no value), con-amp-mt:L02P
- added SV2: (no value), con-amp-mt:L04P
Connections:
- removed net N$61: U$10.CS
- new net CS: SV2-1.S, U$10.CS
- net 0: now also SV1-2.S
- net 5V: now also SV1-1.S
- net CLK: now also SV2-4.S
- net MISO: now also SV2-2.S
- net MOSI: now also SV2-3.S
Changed lines of the file:
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@@
 <part name="R37" library="SparkFun-Resistors" library_urn="urn:adsk.eagle:library:532" deviceset="100KOHM" device="-0603-1/10W-1%" package3d_urn="urn:adsk.eagle:package:39650/1" value="10k"/>
 <part name="R38" library="SparkFun-Resistors" library_urn="urn:adsk.eagle:library:532" deviceset="100KOHM" device="-0603-1/10W-1%" package3d_urn="urn:adsk.eagle:package:39650/1" value="100k"/>
+<part name="SV1" library="con-amp-mt" library_urn="urn:adsk.eagle:library:123" deviceset="L02P" device="" package3d_urn="urn:adsk.eagle:package:5777/1"/>
+<part name="SUPPLY1" library="SparkFun-PowerSymbols" library_urn="urn:adsk.eagle:library:530" deviceset="5V" device=""/>
+<part name="X_1" library="ngspice-simulation" library_urn="urn:adsk.eagle:library:527439" deviceset="GND" device=""/>
+<part name="SV2" library="con-amp-mt" library_urn="urn:adsk.eagle:library:123" deviceset="L04P" device="" package3d_urn="urn:adsk.eagle:package:5780/1"/>
 </parts>
 <sheets>
@@
 <attribute name="NAME" x="157.48" y="105.664" size="1.778" layer="95" font="vector" align="bottom-center"/>
 <attribute name="VALUE" x="157.48" y="102.616" size="1.778" layer="96" font="vector" align="top-center"/>
+</instance>
+<instance part="SV1" gate="-1" x="213.36" y="170.18" smashed="yes">
+<attribute name="NAME" x="212.852" y="171.196" size="1.778" layer="95" rot="R180"/>
+<attribute name="VALUE" x="213.614" y="167.767" size="1.778" layer="96"/>
+</instance>
+<instance part="SV1" gate="-2" x="213.36" y="165.1" smashed="yes">
+<attribute name="NAME" x="212.852" y="166.116" size="1.778" layer="95" rot="R180"/>
+<attribute name="VALUE" x="213.614" y="162.687" size="1.778" layer="96"/>
+</instance>
+<instance part="SUPPLY1" gate="G$1" x="233.68" y="170.18" smashed="yes" rot="R270">
+<attribute name="VALUE" x="236.474" y="170.18" size="1.778" layer="96" rot="R270" align="bottom-center"/>
+</instance>
+<instance part="X_1" gate="G$1" x="236.22" y="162.56" smashed="yes"/>
+<instance part="SV2" gate="-1" x="213.36" y="157.48" smashed="yes">
+<attribute name="NAME" x="212.852" y="158.496" size="1.778" layer="95" rot="R180"/>
+<attribute name="VALUE" x="213.614" y="155.067" size="1.778" layer="96"/>
+</instance>
+<instance part="SV2" gate="-2" x="213.36" y="152.4" smashed="yes">
+<attribute name="NAME" x="212.852" y="153.416" size="1.778" layer="95" rot="R180"/>
+<attribute name="VALUE" x="213.614" y="149.987" size="1.778" layer="96"/>
+</instance>
+<instance part="SV2" gate="-3" x="213.36" y="147.32" smashed="yes">
+<attribute name="NAME" x="212.852" y="148.336" size="1.778" layer="95" rot="R180"/>
+<attribute name="VALUE" x="213.614" y="144.907" size="1.778" layer="96"/>
+</instance>
+<instance part="SV2" gate="-4" x="213.36" y="142.24" smashed="yes">
+<attribute name="NAME" x="212.852" y="143.256" size="1.778" layer="95" rot="R180"/>
+<attribute name="VALUE" x="213.614" y="139.827" size="1.778" layer="96"/>
 </instance>
 </instances>
@@
 <wire x1="172.72" y1="152.4" x2="167.64" y2="152.4" width="0.1524" layer="91"/>
 <junction x="167.64" y="152.4"/>
+</segment>
+<segment>
+<pinref part="X_1" gate="G$1" pin="0"/>
+<wire x1="236.22" y1="162.56" x2="236.22" y2="165.1" width="0.1524" layer="91"/>
+<pinref part="SV1" gate="-2" pin="S"/>
+<wire x1="218.44" y1="165.1" x2="236.22" y2="165.1" width="0.1524" layer="91"/>
 </segment>
 </net>
@@
 <junction x="109.22" y="144.78"/>
 </segment>
+<segment>
+<pinref part="SV1" gate="-1" pin="S"/>
+<wire x1="218.44" y1="170.18" x2="233.68" y2="170.18" width="0.1524" layer="91"/>
+<pinref part="SUPPLY1" gate="G$1" pin="5V"/>
+</segment>
 </net>
 <net name="VCCA" class="0">
@@
 </segment>
 </net>
-<net name="N$61" class="0">
+<net name="CS" class="0">
 <segment>
 <pinref part="U$10" gate="G$1" pin="CS"/>
@@
 <label x="152.4" y="40.64" size="1.778" layer="95"/>
 </segment>
+<segment>
+<wire x1="218.44" y1="157.48" x2="233.68" y2="157.48" width="0.1524" layer="91"/>
+<label x="228.6" y="157.48" size="1.778" layer="95"/>
+<pinref part="SV2" gate="-1" pin="S"/>
+</segment>
 </net>
 <net name="CLK" class="0">
@@
 <label x="152.4" y="35.56" size="1.778" layer="95"/>
 </segment>
+<segment>
+<wire x1="218.44" y1="142.24" x2="233.68" y2="142.24" width="0.1524" layer="91"/>
+<label x="228.6" y="142.24" size="1.778" layer="95"/>
+<pinref part="SV2" gate="-4" pin="S"/>
+</segment>
 </net>
 <net name="MOSI" class="0">
@@
 <label x="96.52" y="35.56" size="1.778" layer="95"/>
 </segment>
+<segment>
+<wire x1="218.44" y1="147.32" x2="233.68" y2="147.32" width="0.1524" layer="91"/>
+<label x="228.6" y="147.32" size="1.778" layer="95"/>
+<pinref part="SV2" gate="-3" pin="S"/>
+</segment>
 </net>
 <net name="MISO" class="0">
@@
 <label x="76.2" y="40.64" size="1.778" layer="95"/>
 </segment>
-</net>
+<segment>
+<wire x1="218.44" y1="152.4" x2="233.68" y2="152.4" width="0.1524" layer="91"/>
+<label x="228.6" y="152.4" size="1.778" layer="95"/>
+<pinref part="SV2" gate="-2" pin="S"/>
+</segment>
+</net>

Commit message: E's systems almost done (only PCB gyro missing)
Parts:
- removed FB1, FB2: 30Ω/1.8A, SparkFun-Coils:FERRITE_BEAD-0603
- removed R14: 2k2, SparkFun-Resistors:0.11OHM-2010-1/2W-1%
- removed R15: 3k3, SparkFun-Resistors:0.11OHM-2010-1/2W-1%
- removed R36: 5.6k, SparkFun-Resistors:5.6KOHM-0603-1/10W-1%
- removed SELF-TEST, SV1: (no value), con-amp-mt:L02P
- removed SV2: (no value), con-amp-mt:L04P
- removed T10: (no value), DC_LOAD_AU:-NPN-SOT23-BEC
- removed U$13, U$15, U$16, U$35: 100nF, Nordic_nRF:CAPACITOR_0603_N
- removed U$33, U$34: 22nF, Nordic_nRF:CAPACITOR_0603_N
- removed U$36: 10nF, Nordic_nRF:CAPACITOR_0603_N
- removed U5: ANALOG_DEVICES_ADXRS646BBGZANALOG_DEVICES_ADXRS646BBGZ_0_0, Analog Devices - ADXRS646BBGZ:ANALOG_DEVICES_ADXRS646BBGZANALOG_DEVICES_ADXRS646BBGZ_0_0
- removed Y1: 16MHz, SparkFun-Clocks:CRYSTAL-26MHZSMD-3.2X2.5
- added J1: (no value), SparkFun-Connectors:CONN_04
- added J2, J3: (no value), SparkFun-Connectors:CONN_02
- added L1, L2: (no value), Wurth_Elektronik_Passive_rev18f:WE-CBA_0805_782853152_HC
- added Q3: FA-128, crystal:FA-128
- added R1: 2k2, SparkFun-Resistors:100KOHM-HORIZ_KIT-1/4W-1%
- added R2: 3k3, SparkFun-Resistors:100KOHM-HORIZ_KIT-1/4W-1%
- added R3: 5k6, SparkFun-Resistors:100KOHM-HORIZ_KIT-1/4W-1%
- added T1: BC846, transistor:BC846
- added U1: ANALOG_DEVICES_ADXRS646BBGZEVAL, Analog Devices - ADXRS646BBGZ-EVAL:ANALOG_DEVICES_ADXRS646BBGZEVAL
- R37: value 10k -> 100k; device SparkFun-Resistors:100KOHM-0603-1/10W-1% -> SparkFun-Resistors:100KOHM-HORIZ_KIT-1/4W-1%
- R38: device SparkFun-Resistors:100KOHM-0603-1/10W-1% -> SparkFun-Resistors:100KOHM-HORIZ_KIT-1/4W-1%
- U$12, U$17, U$18: device Nordic_nRF:CAPACITOR_0603_N -> Nordic_nRF:CAPACITOR_0805_L
Connections:
- removed net N$44: U$10.XTAL2, U$18.2, Y1.2
- removed net N$47: SELF-TEST-2.S, U5A.1_ST2, U5A.2_ST2
- removed net N$52: U$35.1, U5A.1_CP5, U5A.2_CP5
- removed net N$54: U$34.2, U5A.1_CP4, U5A.2_CP4
- removed net N$55: U$34.1, U5A.1_CP3, U5A.2_CP3
- removed net N$56: U$33.2, U5A.1_CP2, U5A.2_CP2
- removed net N$57: U$33.1, U5A.1_CP1, U5A.2_CP1
- new net N$1: J3.1, U1A.ST2
- new net N$2: Q3.3, U$10.XTAL2, U$18.2
- net 0: now also J2.1, L2.1, Q3.2, Q3.4, R2.1, U1B.PGND; no longer FB2.2, R15.1, SV1-2.S, U$16.2, U5B.1_PGND, U5B.2_PGND, Y1.3
- net 5V: now also J2.2, L1.1, R1.2, U1B.VDD; no longer FB1.1, R14.2, SV1-1.S, U$16.1, U5B.1_VDD, U5B.2_VDD
- net CLK: now also J1.1; no longer SV2-4.S
- net CS: now also J1.4; no longer SV2-1.S
- net GND: now also L2.2, U1B.AGND; no longer FB2.1, U$13.2, U$15.2, U$35.2, U5B.1_AGND, U5B.2_AGND
- net MISO: now also J1.3, R3.1; no longer R36.1, SV2-2.S
- net MOSI: now also J1.2; no longer SV2-3.S
- net N$40: now also Q3.1; no longer Y1.1
- net N$42: now also J3.2, U1A.ST1; no longer SELF-TEST-1.S, U5A.1_ST1, U5A.2_ST1
- net N$43: now also T1.C; no longer T10.C
- net N$46: now also T1.B; no longer T10.B
- net N$48: now also U1B.VRATIO; no longer U$13.1, U5B.1_VRATIO, U5B.2_VRATIO
- net N$50: now also R1.1, R2.2; no longer R14.1, R15.2
- net N$53: now also T1.E, U1A.SUMJ; no longer T10.E, U$36.2, U5A.1_SUMJ, U5A.2_SUMJ
- net N$58: now also U1A.RATEOUT; no longer U$36.1, U5A.1_RATEOUT, U5A.2_RATEOUT
- net N$59: now also U1A.TEMP; no longer U5A.1_TEMP, U5A.2_TEMP
- net SDF: now also R3.2; no longer R36.2
- net VCCA: now also L1.2, U1B.AVCC; no longer FB1.2, U$15.1, U5B.1_AVCC, U5B.2_AVCC

Commit message: Final E systems: schematics & PCB's
Connections:
- net CS: now also J1.2; no longer J1.4
- net MOSI: now also J1.4; no longer J1.2
- net N$59: now also U$10.AIN3; no longer U$10.AIN0
