File: 1st iteration/S-multi-PCBs/S-Buck 3.3/irisc.sch (EAGLE design)
At the start: 14 parts, among them IC1 AOZ1284PI

Commit message: Sabina Changes
Parts:
- added BUCK3V1: (no value), SOP65P640X120-17N:BUCK3V3
- added CBIAS: 1 uF, eagle-ltspice:CC1210
- added CBOOT: 0.47 uF, eagle-ltspice:CC1210
- added CFF: 44pF, eagle-ltspice:CC0603
- added CIN1: 0.1uF, Wurth_Elektronik_Passive_Capacitors_rev18b:WCAP-PTHR_6,3X8_870055673001
- added CIN2: 10uF, eagle-ltspice:C
- added COUT4, COUT5, COUT6: 32 uF, eagle-ltspice:CC1812
- added CVCC: 2.2 uF, eagle-ltspice:CC1210
- added CVSS: 22nF, eagle-ltspice:CC1206
- added L2: 22uH, BeagleBone_Blue_R3:INDUCTOR
- added RENB, RENT, RFBT: 1 M, adafruit:FLIPFLOP-RES
- added RFBB: 442 k, adafruit:FLIPFLOP-RES
- added RPG: 10 k, adafruit:FLIPFLOP-RES
- added RT: 200 k, adafruit:FLIPFLOP-RES
- COUT1, COUT2, COUT3: value 32 uF -> 6 uF; device eagle-ltspice:CC1812 -> Wurth_Elektronik_Passive_Capacitors_rev18b:WCAP-CSGP_0805_885012006018_WAVE; SPICEPREFIX (none) -> C
- L1: value 22uH -> (none); device BeagleBone_Blue_R3:INDUCTOR -> inductor-neosid:BS11
Connections:
- new net 3.3V: BUCK3V1.BIAS, CBIAS.1, CFF.1, COUT1.2, COUT2.2, COUT3.2, L1.2, RFBT.2, RPG.1
- new net N$1: BUCK3V1.SW1, BUCK3V1.SW2, CBOOT.1, L1.1
- new net N$12: BUCK3V1.VCC, CVCC.1
- new net N$13: BUCK3V1.PGOOD, RPG.2
- new net N$130: RENB.2, RENT.1
- new net N$14: CBST.1, IC1.LX, L2.1, U$1.P$2
- new net N$2: BUCK3V1.RT, RT.2
- new net N$3: BUCK3V1.SS/TRK, CVSS.1
- new net N$6: BUCK3V1.FB
- new net N$8: CFF.2, RFBB.2, RFBT.1
- new net N$9: BUCK3V1.EN
- new net PGND1: BUCK3V1.PAD, BUCK3V1.PGND1
- new net PGND2: BUCK3V1.AGND, BUCK3V1.PGND2, BUCK3V1.SYNC, CVSS.2, RENB.1, RT.1
- new net VCC1: BUCK3V1.VIN1, BUCK3V1.VIN2, CIN1.1, CIN2.1, RENT.2
- net 5V: now also COUT4.1, COUT5.1, COUT6.1, L2.2; no longer COUT1.1, COUT2.1, COUT3.1, L1.2
- net GND: now also CBIAS.2, CIN1.2, CIN2.2, COUT1.1, COUT2.1, COUT3.1, COUT4.2, COUT5.2, COUT6.2, CVCC.2, RFBB.1; no longer COUT1.2, COUT2.2, COUT3.2
- net N$4: now also BUCK3V1.CBOOT, CBOOT.2; no longer CBST.1, IC1.LX, L1.1, U$1.P$2
Other:
- note added: "BUCK 3V3"
