File: 1st iteration/S-Power/irisc.sch (EAGLE design)
At the start: 4 parts

Commit message: Update irisc.sch
Parts:
- added C10, C11, C12, C4, C5, C6, C7, C8, C9: 0.33µF, SparkFun-Capacitors:0.33UF/330NF-0805-50V-10%
- added U$2, U$3, U$4: (no value), DIP762W50P254L730H410Q6:TRACO
Connections:
- new net N$10: U$2.6
- new net N$11: U$2.4
- new net N$12: U$2.5
- new net N$13: C7.1, C8.1, C9.1, U$3.3
- new net N$14: C7.2, C8.2, C9.2
- new net N$15: U$3.1
- new net N$16: U$3.6
- new net N$17: U$3.4
- new net N$18: U$3.5
- new net N$19: C10.1, C11.1, C12.1, U$4.3
- new net N$20: C10.2, C11.2, C12.2
- new net N$21: U$4.1
- new net N$22: U$4.6
- new net N$23: U$4.4
- new net N$24: U$4.5
- new net N$7: C4.1, C5.1, C6.1, U$2.3
- new net N$8: C4.2, C5.2, C6.2
- new net N$9: U$2.1
- net 2: now also U$2.2, U$3.2, U$4.2
Other:
- note added: "12 V power supply"
- note added: "5 V power supply"
- note removed: "TRACO power components"
